File: Side/side/side.sch (KiCad schematic (older format))
At the start: 3 parts, among them J1 Conn_02x06_Odd_Even, J2 Micro_USB_Breakout, U1 Photon

Commit message: Version 0.1.5 - Various changes, see changelog
Signed-off-by: ray33ee <30669752+ray33ee@users.noreply.github.com>
Parts:
- removed J1: Conn_02x06_Odd_Even, Connector_PinHeader_2.54mm:PinHeader_2x06_P2.54mm_Vertical, symbol Connector_Generic:Conn_02x06_Odd_Even
- added J1: Conn_02x08_Odd_Even, Connector_PinHeader_2.54mm:PinHeader_2x08_P2.54mm_Vertical, symbol Connector_Generic:Conn_02x08_Odd_Even
Connections:
- net +3V3: now also J1.3 (Pin_3)
- net +5V: now also J1.1 (Pin_1)
- net Analogue_0: now also J1.9 (Pin_9)
- net Analogue_1: now also J1.7 (Pin_7)
- net Digital_0: now also U1.17 (D4), J1.13 (Pin_13); no longer U1.15 (D2)
- net Digital_1: now also U1.18 (D5), J1.16 (Pin_16); no longer U1.16 (D3)
- net Digital_2: now also U1.19 (D6), J1.5 (Pin_5); no longer U1.17 (D4)
- net Digital_3: now also U1.20 (D7), J1.14 (Pin_14); no longer U1.18 (D5)
- net Digital_4: now also U1.10 (A2), J1.2 (Pin_2); no longer U1.19 (D6)
- net GND: now also J1.15 (Pin_15)
- net SCL: now also J1.10 (Pin_10)
- net SDA: now also J1.12 (Pin_12)
- net PWM_3: now reaches U1.5 (WKP)
- net PWM_3: now also J1.11 (Pin_11)
- net Digital_5: now reaches U1.9 (A3)
- net Digital_5: now also J1.4 (Pin_4)
- new net PWM_1: J1.8 (Pin_8), U1.15 (D2)
- new net PWM_2: J1.6 (Pin_6), U1.16 (D3)
- no-connect marks 12 -> 8
Changed lines of the file:
@@
 L power:GND #PWR0102
 U 1 1 616EB208
-P 5550 2450
-F 0 "#PWR0102" H 5550 2200 50  0001 C CNN
-F 1 "GND" H 5555 2277 50  0000 C CNN
-F 2 "" H 5550 2450 50  0001 C CNN
-F 3 "" H 5550 2450 50  0001 C CNN
-	1    5550 2450
+P 5350 2450
+F 0 "#PWR0102" H 5350 2200 50  0001 C CNN
+F 1 "GND" H 5355 2277 50  0000 C CNN
+F 2 "" H 5350 2450 50  0001 C CNN
+F 3 "" H 5350 2450 50  0001 C CNN
+	1    5350 2450
 	1    0    0    -1
 $EndComp
@@
 	5550 2350 5950 2350
 Wire Wire Line
-	5550 2450 5950 2450
-Wire Wire Line
 	7300 2350 6700 2350
 Wire Wire Line
@@
 NoConn ~ 5950 2550
 NoConn ~ 5950 2650
-NoConn ~ 5950 2750
 NoConn ~ 5950 2850
-NoConn ~ 5950 3250
-NoConn ~ 5950 3150
-NoConn ~ 5950 3050
 NoConn ~ 5950 2950
 Wire Wire Line
@@
 	1    0    0    -1
 $EndComp
-$Comp
-L Connector_Generic:Conn_02x06_Odd_Even J1
-U 1 1 616F1D95
-P 8600 3700
-F 0 "J1" H 8650 4117 50  0000 C CNN
-F 1 "Conn_02x06_Odd_Even" H 8650 4026 50  0000 C CNN
-F 2 "Connector_PinHeader_2.54mm:PinHeader_2x06_P2.54mm_Vertical" H 8600 3700 50  0001 C CNN
-F 3 "~" H 8600 3700 50  0001 C CNN
-	1    8600 3700
-	1    0    0    -1
-$EndComp
-Wire Wire Line
-	8900 4000 9350 4000
-Wire Wire Line
-	8900 3900 9350 3900
-Wire Wire Line
-	9350 3600 8900 3600
-Wire Wire Line
-	9350 3500 8900 3500
-Text Label 9350 4000 2    50   ~ 0
+Wire Wire Line
+	8900 3850 9350 3850
+Wire Wire Line
+	8900 3750 9350 3750
+Wire Wire Line
+	9350 3450 8900 3450
+Wire Wire Line
+	9350 3350 8900 3350
+Text Label 9350 3850 2    50   ~ 0
 SDA
-Text Label 9350 3900 2    50   ~ 0
+Text Label 9350 3750 2    50   ~ 0
 SCL
-Text Label 9350 3600 2    50   ~ 0
+Text Label 9350 4050 2    50   ~ 0
+Digital_1
+Wire Wire Line
+	9350 3650 8900 3650
+Wire Wire Line
+	9350 3550 8900 3550
+Text Label 9350 3650 2    50   ~ 0
+PWM_1
+Text Label 9350 3550 2    50   ~ 0
+PWM_2
+Wire Wire Line
+	7950 3750 8400 3750
+Wire Wire Line
+	7950 3650 8400 3650
+Text Label 7950 3650 0    50   ~ 0
+Analogue_1
+Text Label 7950 3750 0    50   ~ 0
+Analogue_0
+Wire Wire Line
+	7950 3550 8400 3550
+Text Label 7950 3550 0    50   ~ 0
 Digital_2
-Text Label 9350 3500 2    50   ~ 0
-Digital_3
-Wire Wire Line
-	9350 3800 8900 3800
-Wire Wire Line
-	9350 3700 8900 3700
-Text Label 9350 3800 2    50   ~ 0
-Digital_0
-Text Label 9350 3700 2    50   ~ 0
-Digital_1
-Wire Wire Line
-	7950 4000 8400 4000
-Wire Wire Line
-	7950 3900 8400 3900
-Text Label 7950 3900 0    50   ~ 0
-Analogue_1
-Text Label 7950 4000 0    50   ~ 0
-Analogue_0
-Wire Wire Line
-	7950 3800 8400 3800
-Text Label 7950 3800 0    50   ~ 0
-Digital_4
 $Comp
 L power:GND #PWR0107
 U 1 1 616F5568
-P 7750 3700
-F 0 "#PWR0107" H 7750 3450 50  0001 C CNN
-F 1 "GND" H 7755 3527 50  0000 C CNN
-F 2 "" H 7750 3700 50  0001 C CNN
-F 3 "" H 7750 3700 50  0001 C CNN
-	1    7750 3700
+P 7750 4050
+F 0 "#PWR0107" H 7750 3800 50  0001 C CNN
+F 1 "GND" H 7755 3877 50  0000 C CNN
+F 2 "" H 7750 4050 50  0001 C CNN
+F 3 "" H 7750 4050 50  0001 C CNN
+	1    7750 4050
 	1    0    0    -1
 $EndComp
@@
 L power:+5V #PWR0108
 U 1 1 616F5A38
-P 8050 3500
-F 0 "#PWR0108" H 8050 3350 50  0001 C CNN
-F 1 "+5V" H 8065 3673 50  0000 C CNN
-F 2 "" H 8050 3500 50  0001 C CNN
-F 3 "" H 8050 3500 50  0001 C CNN
-	1    8050 3500
+P 8050 3350
+F 0 "#PWR0108" H 8050 3200 50  0001 C CNN
+F 1 "+5V" H 8065 3523 50  0000 C CNN
+F 2 "" H 8050 3350 50  0001 C CNN
+F 3 "" H 8050 3350 50  0001 C CNN
+	1    8050 3350
 	1    0    0    -1
 $EndComp
@@
 L power:+3.3V #PWR0109
 U 1 1 616F5B83
-P 7800 3500
-F 0 "#PWR0109" H 7800 3350 50  0001 C CNN
-F 1 "+3.3V" H 7815 3673 50  0000 C CNN
-F 2 "" H 7800 3500 50  0001 C CNN
-F 3 "" H 7800 3500 50  0001 C CNN
-	1    7800 3500
-	1    0    0    -1
-$EndComp
-Wire Wire Line
-	7750 3700 8400 3700
-Wire Wire Line
-	8400 3600 7800 3600
-Wire Wire Line
-	7800 3600 7800 3500
-Wire Wire Line
-	8050 3500 8400 3500
+P 7800 3350
+F 0 "#PWR0109" H 7800 3200 50  0001 C CNN
+F 1 "+3.3V" H 7815 3523 50  0000 C CNN
+F 2 "" H 7800 3350 50  0001 C CNN
+F 3 "" H 7800 3350 50  0001 C CNN
+	1    7800 3350
+	1    0    0    -1
+$EndComp
+Wire Wire Line
+	7750 4050 8400 4050
+Wire Wire Line
+	8400 3450 7800 3450
+Wire Wire Line
+	7800 3450 7800 3350
+Wire Wire Line
+	8050 3350 8400 3350
 Text Label 7150 3150 2    50   ~ 0
-Digital_1
-Text Label 7150 3250 2    50   ~ 0
-Digital_0
+PWM_2
 Wire Wire Line
 	7150 3150 6700 3150
@@
 	7150 3250 6700 3250
 Text Label 7150 2850 2    50   ~ 0
-Digital_4
+Digital_2
 Text Label 7150 2950 2    50   ~ 0
-Digital_3
+Digital_1
 Text Label 7150 3050 2    50   ~ 0
-Digital_2
+Digital_0
 Text Label 7150 3350 2    50   ~ 0
 SCL
@@
 NoConn ~ 6700 2550
 NoConn ~ 6700 2450
-NoConn ~ 6700 2750
 $Comp
 L Device:Photon U1
@@
 Wire Wire Line
 	7800 2800 8400 2800
+$Comp
+L Connector_Generic:Conn_02x08_Odd_Even J1
+U 1 1 616EE07C
+P 8600 3650
+F 0 "J1" H 8650 4167 50  0000 C CNN
+F 1 "Conn_02x08_Odd_Even" H 8650 4076 50  0000 C CNN
+F 2 "Connector_PinHeader_2.54mm:PinHeader_2x08_P2.54mm_Vertical" H 8600 3650 50  0001 C CNN
+F 3 "~" H 8600 3650 50  0001 C CNN
+	1    8600 3650
+	1    0    0    -1
+$EndComp
+Text Label 7150 2750 2    50   ~ 0
+Digital_3
+Wire Wire Line
+	7150 2750 6700 2750
+Text Label 9350 3950 2    50   ~ 0
+Digital_3
+Wire Wire Line
+	9350 3950 8900 3950
+Text Label 5500 3250 0    50   ~ 0
+Digital_4
+Wire Wire Line
+	5500 3250 5950 3250
+Text Label 5500 3150 0    50   ~ 0
+Digital_5
+Wire Wire Line
+	5500 3150 5950 3150
+Text Label 5500 2750 0    50   ~ 0
+PWM_3
+Wire Wire Line
+	5500 2750 5950 2750
+Text Label 9350 3350 2    50   ~ 0
+Digital_4
+Wire Wire Line
+	9350 4050 8900 4050
+Text Label 9350 3450 2    50   ~ 0
+Digital_5
+Wire Wire Line
+	7950 3950 8400 3950
+Text Label 7150 3250 2    50   ~ 0
+PWM_1
+Wire Wire Line
+	5350 2450 5950 2450
+NoConn ~ 5950 3050
+Wire Wire Line
+	7950 3850 8400 3850
+Text Label 7950 3850 0    50   ~ 0
+PWM_3
+Text Label 7950 3950 0    50   ~ 0
+Digital_0
 $EndSCHEMATC

Commit message: Version 0.1.7 - Various changes, see changelog
Signed-off-by: ray33ee <30669752+ray33ee@users.noreply.github.com>
Parts:
- added R1, R2: 10k, Resistor_SMD:R_1206_3216Metric_Pad1.30x1.75mm_HandSolder, symbol Device:R
Connections:
- net +3V3: now also R1.1, R2.1
- net SCL: now also R1.2
- net SDA: now also R2.2
Other:
- moved on the sheet: J1, J2
Changed lines of the file:
@@
 L power:+3.3V #PWR0103
 U 1 1 616EB387
-P 7300 2350
-F 0 "#PWR0103" H 7300 2200 50  0001 C CNN
-F 1 "+3.3V" H 7315 2523 50  0000 C CNN
-F 2 "" H 7300 2350 50  0001 C CNN
-F 3 "" H 7300 2350 50  0001 C CNN
-	1    7300 2350
+P 8000 2350
+F 0 "#PWR0103" H 8000 2200 50  0001 C CNN
+F 1 "+3.3V" H 8015 2523 50  0000 C CNN
+F 2 "" H 8000 2350 50  0001 C CNN
+F 3 "" H 8000 2350 50  0001 C CNN
+	1    8000 2350
 	1    0    0    -1
 $EndComp
@@
 	5550 2350 5950 2350
 Wire Wire Line
-	7300 2350 6700 2350
-Wire Wire Line
 	6700 2650 7300 2650
 NoConn ~ 5950 2550
@@
 L power:GND #PWR0105
 U 1 1 616F01C4
-P 7800 2400
-F 0 "#PWR0105" H 7800 2150 50  0001 C CNN
-F 1 "GND" H 7805 2227 50  0000 C CNN
-F 2 "" H 7800 2400 50  0001 C CNN
-F 3 "" H 7800 2400 50  0001 C CNN
-	1    7800 2400
+P 9050 2300
+F 0 "#PWR0105" H 9050 2050 50  0001 C CNN
+F 1 "GND" H 9055 2127 50  0000 C CNN
+F 2 "" H 9050 2300 50  0001 C CNN
+F 3 "" H 9050 2300 50  0001 C CNN
+	1    9050 2300
 	1    0    0    -1
 $EndComp
@@
 L power:+5V #PWR0106
 U 1 1 616F0805
-P 7800 2800
-F 0 "#PWR0106" H 7800 2650 50  0001 C CNN
-F 1 "+5V" H 7815 2973 50  0000 C CNN
-F 2 "" H 7800 2800 50  0001 C CNN
-F 3 "" H 7800 2800 50  0001 C CNN
-	1    7800 2800
-	1    0    0    -1
-$EndComp
-Wire Wire Line
-	8900 3850 9350 3850
-Wire Wire Line
-	8900 3750 9350 3750
-Wire Wire Line
-	9350 3450 8900 3450
-Wire Wire Line
-	9350 3350 8900 3350
-Text Label 9350 3850 2    50   ~ 0
+P 9050 2700
+F 0 "#PWR0106" H 9050 2550 50  0001 C CNN
+F 1 "+5V" H 9065 2873 50  0000 C CNN
+F 2 "" H 9050 2700 50  0001 C CNN
+F 3 "" H 9050 2700 50  0001 C CNN
+	1    9050 2700
+	1    0    0    -1
+$EndComp
+Wire Wire Line
+	10000 3850 10450 3850
+Wire Wire Line
+	10000 3750 10450 3750
+Wire Wire Line
+	10450 3450 10000 3450
+Wire Wire Line
+	10450 3350 10000 3350
+Text Label 10450 3850 2    50   ~ 0
 SDA
-Text Label 9350 3750 2    50   ~ 0
+Text Label 10450 3750 2    50   ~ 0
 SCL
-Text Label 9350 4050 2    50   ~ 0
+Text Label 10450 4050 2    50   ~ 0
 Digital_1
 Wire Wire Line
-	9350 3650 8900 3650
-Wire Wire Line
-	9350 3550 8900 3550
-Text Label 9350 3650 2    50   ~ 0
+	10450 3650 10000 3650
+Wire Wire Line
+	10450 3550 10000 3550
+Text Label 10450 3650 2    50   ~ 0
 PWM_1
-Text Label 9350 3550 2    50   ~ 0
+Text Label 10450 3550 2    50   ~ 0
 PWM_2
 Wire Wire Line
-	7950 3750 8400 3750
-Wire Wire Line
-	7950 3650 8400 3650
-Text Label 7950 3650 0    50   ~ 0
+	9050 3750 9500 3750
+Wire Wire Line
+	9050 3650 9500 3650
+Text Label 9050 3650 0    50   ~ 0
 Analogue_1
-Text Label 7950 3750 0    50   ~ 0
+Text Label 9050 3750 0    50   ~ 0
 Analogue_0
 Wire Wire Line
-	7950 3550 8400 3550
-Text Label 7950 3550 0    50   ~ 0
+	9050 3550 9500 3550
+Text Label 9050 3550 0    50   ~ 0
 Digital_2
 $Comp
 L power:GND #PWR0107
 U 1 1 616F5568
-P 7750 4050
-F 0 "#PWR0107" H 7750 3800 50  0001 C CNN
-F 1 "GND" H 7755 3877 50  0000 C CNN
-F 2 "" H 7750 4050 50  0001 C CNN
-F 3 "" H 7750 4050 50  0001 C CNN
-	1    7750 4050
+P 8850 4050
+F 0 "#PWR0107" H 8850 3800 50  0001 C CNN
+F 1 "GND" H 8855 3877 50  0000 C CNN
+F 2 "" H 8850 4050 50  0001 C CNN
+F 3 "" H 8850 4050 50  0001 C CNN
+	1    8850 4050
 	1    0    0    -1
 $EndComp
@@
 L power:+5V #PWR0108
 U 1 1 616F5A38
-P 8050 3350
-F 0 "#PWR0108" H 8050 3200 50  0001 C CNN
-F 1 "+5V" H 8065 3523 50  0000 C CNN
-F 2 "" H 8050 3350 50  0001 C CNN
-F 3 "" H 8050 3350 50  0001 C CNN
-	1    8050 3350
+P 9150 3350
+F 0 "#PWR0108" H 9150 3200 50  0001 C CNN
+F 1 "+5V" H 9165 3523 50  0000 C CNN
+F 2 "" H 9150 3350 50  0001 C CNN
+F 3 "" H 9150 3350 50  0001 C CNN
+	1    9150 3350
 	1    0    0    -1
 $EndComp
@@
 L power:+3.3V #PWR0109
 U 1 1 616F5B83
-P 7800 3350
-F 0 "#PWR0109" H 7800 3200 50  0001 C CNN
-F 1 "+3.3V" H 7815 3523 50  0000 C CNN
-F 2 "" H 7800 3350 50  0001 C CNN
-F 3 "" H 7800 3350 50  0001 C CNN
-	1    7800 3350
-	1    0    0    -1
-$EndComp
-Wire Wire Line
-	7750 4050 8400 4050
-Wire Wire Line
-	8400 3450 7800 3450
-Wire Wire Line
-	7800 3450 7800 3350
-Wire Wire Line
-	8050 3350 8400 3350
+P 8900 3350
+F 0 "#PWR0109" H 8900 3200 50  0001 C CNN
+F 1 "+3.3V" H 8915 3523 50  0000 C CNN
+F 2 "" H 8900 3350 50  0001 C CNN
+F 3 "" H 8900 3350 50  0001 C CNN
+	1    8900 3350
+	1    0    0    -1
+$EndComp
+Wire Wire Line
+	8850 4050 9500 4050
+Wire Wire Line
+	9500 3450 8900 3450
+Wire Wire Line
+	8900 3450 8900 3350
+Wire Wire Line
+	9150 3350 9500 3350
 Text Label 7150 3150 2    50   ~ 0
 PWM_2
@@
 Text Label 7150 3050 2    50   ~ 0
 Digital_0
-Text Label 7150 3350 2    50   ~ 0
+Text Label 8450 3350 2    50   ~ 0
 SCL
-Text Label 7150 3450 2    50   ~ 0
+Text Label 8450 3450 2    50   ~ 0
 SDA
 Wire Wire Line
@@
 Wire Wire Line
 	7150 3050 6700 3050
-Wire Wire Line
-	6700 3350 7150 3350
-Wire Wire Line
-	6700 3450 7150 3450
 NoConn ~ 6700 2550
 NoConn ~ 6700 2450
@@
 D-
 Wire Wire Line
-	8400 2600 7950 2600
-Wire Wire Line
-	8400 2700 7950 2700
-Text Label 7950 2600 0    50   ~ 0
+	9650 2500 9200 2500
+Wire Wire Line
+	9650 2600 9200 2600
+Text Label 9200 2500 0    50   ~ 0
 D+
-Text Label 7950 2700 0    50   ~ 0
+Text Label 9200 2600 0    50   ~ 0
 D-
 $Comp
 L Connector_Generic:Conn_01x05 J2
 U 1 1 616EC106
-P 8600 2600
-F 0 "J2" H 8680 2642 50  0000 L CNN
-F 1 "Micro_USB_Breakout" H 8680 2551 50  0000 L CNN
-F 2 "Socket:Adafruit_Micro_USB_Breakout_copy" H 8680 2505 50  0001 L CNN
-F 3 "~" H 8600 2600 50  0001 C CNN
-	1    8600 2600
-	1    0    0    -1
-$EndComp
-NoConn ~ 8400 2500
-Wire Wire Line
-	8400 2400 7800 2400
-Wire Wire Line
-	7800 2800 8400 2800
+P 9850 2500
+F 0 "J2" H 9930 2542 50  0000 L CNN
+F 1 "Micro_USB_Breakout" H 9930 2451 50  0000 L CNN
+F 2 "Socket:Adafruit_Micro_USB_Breakout_copy" H 9930 2405 50  0001 L CNN
+F 3 "~" H 9850 2500 50  0001 C CNN
+	1    9850 2500
+	1    0    0    -1
+$EndComp
+NoConn ~ 9650 2400
+Wire Wire Line
+	9650 2300 9050 2300
+Wire Wire Line
+	9050 2700 9650 2700
 $Comp
 L Connector_Generic:Conn_02x08_Odd_Even J1
 U 1 1 616EE07C
-P 8600 3650
-F 0 "J1" H 8650 4167 50  0000 C CNN
-F 1 "Conn_02x08_Odd_Even" H 8650 4076 50  0000 C CNN
-F 2 "Connector_PinHeader_2.54mm:PinHeader_2x08_P2.54mm_Vertical" H 8600 3650 50  0001 C CNN
-F 3 "~" H 8600 3650 50  0001 C CNN
-	1    8600 3650
+P 9700 3650
+F 0 "J1" H 9750 4167 50  0000 C CNN
+F 1 "Conn_02x08_Odd_Even" H 9750 4076 50  0000 C CNN
+F 2 "Connector_PinHeader_2.54mm:PinHeader_2x08_P2.54mm_Vertical" H 9700 3650 50  0001 C CNN
+F 3 "~" H 9700 3650 50  0001 C CNN
+	1    9700 3650
 	1    0    0    -1
 $EndComp
@@
 Wire Wire Line
 	7150 2750 6700 2750
-Text Label 9350 3950 2    50   ~ 0
+Text Label 10450 3950 2    50   ~ 0
 Digital_3
 Wire Wire Line
-	9350 3950 8900 3950
+	10450 3950 10000 3950
 Text Label 5500 3250 0    50   ~ 0
 Digital_4
@@
 Wire Wire Line
 	5500 2750 5950 2750
-Text Label 9350 3350 2    50   ~ 0
+Text Label 10450 3350 2    50   ~ 0
 Digital_4
 Wire Wire Line
-	9350 4050 8900 4050
-Text Label 9350 3450 2    50   ~ 0
+	10450 4050 10000 4050
+Text Label 10450 3450 2    50   ~ 0
 Digital_5
 Wire Wire Line
-	7950 3950 8400 3950
+	9050 3950 9500 3950
 Text Label 7150 3250 2    50   ~ 0
 PWM_1
@@
 NoConn ~ 5950 3050
 Wire Wire Line
-	7950 3850 8400 3850
-Text Label 7950 3850 0    50   ~ 0
+	9050 3850 9500 3850
+Text Label 9050 3850 0    50   ~ 0
 PWM_3
-Text Label 7950 3950 0    50   ~ 0
+Text Label 9050 3950 0    50   ~ 0
 Digital_0
+$Comp
+L Device:R R1
+U 1 1 6170EB0B
+P 7750 3050
+F 0 "R1" H 7820 3096 50  0000 L CNN
+F 1 "10k" H 7820 3005 50  0000 L CNN
+F 2 "Resistor_SMD:R_1206_3216Metric_Pad1.30x1.75mm_HandSolder" V 7680 3050 50  0001 C CNN
+F 3 "~" H 7750 3050 50  0001 C CNN
+	1    7750 3050
+	1    0    0    -1
+$EndComp
+$Comp
+L Device:R R2
+U 1 1 6170F2DF
+P 8000 3050
+F 0 "R2" H 8070 3096 50  0000 L CNN
+F 1 "10k" H 8070 3005 50  0000 L CNN
+F 2 "Resistor_SMD:R_1206_3216Metric_Pad1.30x1.75mm_HandSolder" V 7930 3050 50  0001 C CNN
+F 3 "~" H 8000 3050 50  0001 C CNN
+	1    8000 3050
+	1    0    0    -1
+$EndComp
+Wire Wire Line
+	7750 3200 7750 3350
+Connection ~ 7750 3350
+Wire Wire Line
+	7750 3350 8450 3350
+Wire Wire Line
+	8000 3200 8000 3450
+Connection ~ 8000 3450
+Wire Wire Line
+	8000 3450 8450 3450
+Wire Wire Line
+	6700 3350 7750 3350
+Wire Wire Line
+	6700 3450 8000 3450
+Wire Wire Line
+	7750 2350 7750 2900
+Wire Wire Line
+	7750 2350 8000 2350
+Wire Wire Line
+	8000 2350 8000 2900
+Connection ~ 7750 2350
+Connection ~ 8000 2350
+Wire Wire Line
+	6700 2350 7750 2350
 $EndSCHEMATC

Commit message: Version 0.1.14 - Various changes, see changelog
Signed-off-by: ray33ee <30669752+ray33ee@users.noreply.github.com>
Connections:
- net Digital_1: now also U1.4 (RX); no longer U1.18 (D5)
- net Digital_2: now also U1.6 (DAC); no longer U1.19 (D6)
- net Digital_3: now also U1.7 (A5); no longer U1.20 (D7)
- net PWM_2: now also U1.8 (A4); no longer U1.16 (D3)
Changed lines of the file:
@@
 	6700 2650 7300 2650
 NoConn ~ 5950 2550
-NoConn ~ 5950 2650
-NoConn ~ 5950 2850
-NoConn ~ 5950 2950
 Wire Wire Line
 	5500 3450 5950 3450
@@
 Wire Wire Line
 	9150 3350 9500 3350
-Text Label 7150 3150 2    50   ~ 0
-PWM_2
-Wire Wire Line
-	7150 3150 6700 3150
 Wire Wire Line
 	7150 3250 6700 3250
-Text Label 7150 2850 2    50   ~ 0
+Text Label 5500 2850 0    50   ~ 0
 Digital_2
-Text Label 7150 2950 2    50   ~ 0
+Text Label 5500 2650 0    50   ~ 0
 Digital_1
 Text Label 7150 3050 2    50   ~ 0
@@
 SDA
 Wire Wire Line
-	7150 2850 6700 2850
-Wire Wire Line
-	7150 2950 6700 2950
+	5500 2850 5950 2850
+Wire Wire Line
+	5500 2650 5950 2650
 Wire Wire Line
 	7150 3050 6700 3050
@@
 	1    0    0    -1
 $EndComp
-Text Label 7150 2750 2    50   ~ 0
+Text Label 5500 2950 0    50   ~ 0
 Digital_3
 Wire Wire Line
-	7150 2750 6700 2750
+	5500 2950 5950 2950
 Text Label 10450 3950 2    50   ~ 0
 Digital_3
@@
 Wire Wire Line
 	5350 2450 5950 2450
-NoConn ~ 5950 3050
 Wire Wire Line
 	9050 3850 9500 3850
@@
 Wire Wire Line
 	6700 2350 7750 2350
+Wire Wire Line
+	5500 3050 5950 3050
+Text Label 5500 3050 0    50   ~ 0
+PWM_2
+NoConn ~ 6700 3150
+NoConn ~ 6700 2750
+NoConn ~ 6700 2850
+NoConn ~ 6700 2950
 $EndSCHEMATC
