File: Side/side/side.kicad_pcb (KiCad board)
At the start: 2 copper layers, 28.5 x 51.8 mm, 3 parts, among them J1 Conn_02x06_Odd_Even, J2 Micro_USB_Breakout, U1 Photon

Commit message: Version 0.1.5 - Various changes, see changelog
Signed-off-by: ray33ee <30669752+ray33ee@users.noreply.github.com>
Parts:
- J1: value Conn_02x06_Odd_Even -> Conn_02x08_Odd_Even; footprint Connector_PinHeader_2.54mm:PinHeader_2x06_P2.54mm_Vertical -> Connector_PinHeader_2.54mm:PinHeader_2x08_P2.54mm_Vertical
- moved J1 3.84 mm to (199.3, 94.9)
- moved J2 3.00 mm to (206.4, 97.7)
Connections:
- J1 pad 11: /Analogue_0 -> /PWM_3
- J1 pad 2: /Digital_3 -> /Digital_4
- J1 pad 4: /Digital_2 -> /Digital_5
- J1 pad 5: GND -> /Digital_2
- J1 pad 6: /Digital_1 -> /PWM_2
- J1 pad 7: /Digital_4 -> /Analogue_1
- J1 pad 8: /Digital_0 -> /PWM_1
- J1 pad 9: /Analogue_1 -> /Analogue_0
- U1 pad 10: Net-(U1-Pad10) -> /Digital_4
- U1 pad 15: /Digital_0 -> /PWM_1
- U1 pad 16: /Digital_1 -> /PWM_2
- U1 pad 17: /Digital_2 -> /Digital_0
- U1 pad 18: /Digital_3 -> /Digital_1
- U1 pad 19: /Digital_4 -> /Digital_2
- U1 pad 20: Net-(U1-Pad20) -> /Digital_3
- U1 pad 5: Net-(U1-Pad5) -> /PWM_3
- U1 pad 9: Net-(U1-Pad9) -> /Digital_5
Routing:
- net /PWM_2: track 0.00 -> 46.4 mm, vias 0 -> 1
- net /PWM_1: track 0.00 -> 45.7 mm, vias 0 -> 1
- net /Digital_5: track 0.00 -> 38.7 mm, vias 0 -> 1
- net /PWM_3: track 0.00 -> 37.3 mm, vias 0 -> 1
- net /Digital_3: track 50.1 -> 25.9 mm
- net /Digital_0: track 46.2 -> 31.3 mm
- net /Digital_1: track 46.7 -> 32.8 mm
- net /Digital_2: track 49.0 -> 37.1 mm
- net /Analogue_1: track 57.9 -> 50.1 mm
- net GND: track 45.3 -> 52.6 mm
- net +5V: track 41.5 -> 34.1 mm, vias 3 -> 2
- net /Analogue_0: track 60.3 -> 53.0 mm
- net /D-: track 14.9 -> 12.0 mm
- net /SCL: track 55.7 -> 52.9 mm, vias 1 -> 3
- net /Digital_4: track 35.7 -> 38.2 mm
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Other:
- board text added: "Valve Controller Side v1.1|William RJ Cooper|github.com/ray33ee"
- board text removed: "Valve Controller Side v1.0|William RJ Cooper|github.com/ray33ee"

Commit message: Version 0.1.7 - Various changes, see changelog
Signed-off-by: ray33ee <30669752+ray33ee@users.noreply.github.com>
Parts:
- added R1: 10k, Resistor_SMD:R_1206_3216Metric_Pad1.30x1.75mm_HandSolder, B.Cu at (211.8, 122.8)
- added R2: 10k, Resistor_SMD:R_1206_3216Metric_Pad1.30x1.75mm_HandSolder, B.Cu at (214.5, 122.8)
- moved J1 1.00 mm to (199.3, 93.9)
- moved J2 1.00 mm to (206.4, 96.7)
Routing:
- net +3V3: track 26.3 -> 45.8 mm, vias 1 -> 2
- net /SCL: track 52.9 -> 65.2 mm, vias 3 -> 5
- net /SDA: track 50.9 -> 58.8 mm
- net +5V: track 34.1 -> 35.5 mm
- net /PWM_3: track 37.3 -> 38.3 mm
- net /PWM_2: track 46.4 -> 47.4 mm
- net /PWM_1: track 45.7 -> 46.7 mm
- net /Digital_5: track 38.7 -> 39.7 mm
- net /Digital_3: track 25.9 -> 26.9 mm
- net /Digital_2: track 37.1 -> 38.1 mm
- net /Digital_1: track 32.8 -> 33.8 mm
- net /Digital_0: track 31.3 -> 32.3 mm
- net /D-: track 12.0 -> 13.0 mm
- net /D+: track 14.7 -> 15.7 mm
- net /Analogue_0: track 53.0 -> 54.0 mm
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
Commit message: Version 0.1.14 - Various changes, see changelog
Signed-off-by: ray33ee <30669752+ray33ee@users.noreply.github.com>
Connections:
- U1 pad 16: /PWM_2 -> Net-(U1-Pad16)
- U1 pad 18: /Digital_1 -> Net-(U1-Pad18)
- U1 pad 19: /Digital_2 -> Net-(U1-Pad19)
- U1 pad 20: /Digital_3 -> Net-(U1-Pad20)
- U1 pad 4: Net-(U1-Pad4) -> /Digital_1
- U1 pad 6: Net-(U1-Pad6) -> /Digital_2
- U1 pad 7: Net-(U1-Pad7) -> /Digital_3
- U1 pad 8: Net-(U1-Pad8) -> /PWM_2
Routing:
- net /Digital_3: track 26.9 -> 48.4 mm
- net Net-(U1-Pad18): track 0.00 -> 18.4 mm, vias 0 -> 1
- net /Digital_1: track 33.8 -> 44.6 mm, vias 1 -> 3
- net /Digital_2: track 38.1 -> 30.3 mm
- net /PWM_2: track 47.4 -> 39.7 mm
- net +5V: vias 2 -> 1

Commit message: Version 0.1.15 - Various changes, see changelog
Signed-off-by: ray33ee <30669752+ray33ee@users.noreply.github.com>
Routing:
- net Net-(U1-Pad18): track 18.4 -> 0.00 mm, vias 1 -> 0
- net /PWM_1: track 46.7 -> 50.6 mm
- net /PWM_2: track 39.7 -> 39.2 mm
- net +5V: vias 1 -> 3
Other:
- board text added: "Valve Controller Side v1.2|William RJ Cooper|github.com/ray33ee"
- board text removed: "Valve Controller Side v1.1|William RJ Cooper|github.com/ray33ee"
