File: Top/top/top.kicad_pcb (KiCad board)
At the start: 2 copper layers, 45 x 45 mm, 3 parts

Commit message: Version 0.1.5 - Various changes, see changelog
Signed-off-by: ray33ee <30669752+ray33ee@users.noreply.github.com>
Parts:
- added D1: LED_RBGA, LED_SMD:LED_Cree-PLCC4_3.2x2.88mm_CCW_Hand_Solder, F.Cu at (139.9, 93.3)
- added J1: Conn_02x08_Odd_Even, Connector_PinHeader_2.54mm:PinHeader_2x08_P2.54mm_Vertical, F.Cu at (130.2, 75.2)
- added J2: Conn_01x10_Female, Connector_PinHeader_2.54mm:PinHeader_1x10_P2.54mm_Vertical, F.Cu at (145.7, 73.5)
- added J3: Header, Connector_PinHeader_2.54mm:PinHeader_1x04_P2.54mm_Vertical, F.Cu at (125.5, 107.1)
- added J4: JST Connector, Connector_JST:JST_SH_SM04B-SRSS-TB_1x04-1MP_P1.00mm_Horizontal, F.Cu at (141.4, 105.3)
- added R1: 680, Resistor_SMD:R_1206_3216Metric_Pad1.30x1.75mm_HandSolder, F.Cu at (134.0, 91.4)
- added R2: 470, Resistor_SMD:R_1206_3216Metric_Pad1.30x1.75mm_HandSolder, F.Cu at (145.6, 94.2)
- added R3: 470, Resistor_SMD:R_1206_3216Metric_Pad1.30x1.75mm_HandSolder, F.Cu at (134.0, 95.4)
Routing:
- net +3V3: track 0.00 -> 19.3 mm
- net GND: track 0.00 -> 17.4 mm
- net /SCL: track 0.00 -> 15.5 mm
- net /SDA: track 0.00 -> 13.6 mm
- net /B: track 0.00 -> 3.68 mm
- net /R: track 0.00 -> 3.60 mm
- net /G: track 0.00 -> 2.93 mm

Commit message: Version 0.1.7 - Various changes, see changelog
Signed-off-by: ray33ee <30669752+ray33ee@users.noreply.github.com>
Parts:
- removed REF** (x3): MountingHole_2.5mm, MountingHole:MountingHole_2.5mm
- added MH1: GenericMountingHole, MountingHole:GenericMountingHole, F.Cu at (155.8, 111.8)
- added MH2: GenericMountingHole, MountingHole:GenericMountingHole, F.Cu at (138.2, 142.1)
- added MH3: GenericMountingHole, MountingHole:GenericMountingHole, F.Cu at (175.3, 145.7)
- moved J2 64.4 mm to (177.6, 129.4), turned to 225.4 degrees
- moved J3 48.2 mm to (147.5, 150.0), turned to 70 degrees
- moved J4 45.2 mm to (166.9, 142.6)
- moved R1 44.7 mm to (153.0, 131.9)
- moved R2 43.9 mm to (164.5, 133.8)
- moved D1 43.8 mm to (158.2, 133.1)
- moved J1 43.3 mm to (146.6, 115.3), turned to 327.2 degrees
- moved R3 43.3 mm to (153.0, 134.3)
Routing:
- net GND: track 17.4 -> 86.2 mm
- net /Enabled_Controlled: track 0.00 -> 45.5 mm, vias 0 -> 1
- net +3V3: track 19.3 -> 62.4 mm, vias 0 -> 2
- net +5V: track 0.00 -> 40.1 mm, vias 0 -> 1
- net /SDA: track 13.6 -> 52.1 mm, vias 0 -> 2
- net /PushButton: track 0.00 -> 38.4 mm, vias 0 -> 1
- net /SCL: track 15.5 -> 53.2 mm, vias 0 -> 4
- net /Coil_A1: track 0.00 -> 36.4 mm, vias 0 -> 1
- net /Coil_B2: track 0.00 -> 35.3 mm, vias 0 -> 2
- net /Diff_P1: track 0.00 -> 31.1 mm, vias 0 -> 1
- net /LED_Green: track 0.00 -> 30.4 mm, vias 0 -> 2
- net /Diff_P2: track 0.00 -> 27.3 mm, vias 0 -> 1
- net /Coil_A2: track 0.00 -> 18.9 mm, vias 0 -> 1
- net /LED_Blue: track 0.00 -> 17.5 mm, vias 0 -> 2
- net /LED_Red: track 0.00 -> 16.8 mm, vias 0 -> 2
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Other:
- net class Default: clearance 0.2 -> 0.127; trace_width 0.25 -> 0.15; via_dia 0.8 -> 0.4; via_drill 0.4 -> 0.2
- net class High Current added: clearance 0.15, trace_width 0.6, via_dia 0.6, via_drill 0.3
- rule trace_clearance: 0.2 -> 0.127
- rule trace_min: 0.2 -> 0.127
- rule via_min_drill: 0.3 -> 0.2

Commit message: Version 0.1.8 - Various changes, see changelog
Signed-off-by: ray33ee <30669752+ray33ee@users.noreply.github.com>
Parts:
- moved MH2 1.05 mm to (137.9, 141.1)
Other:
- board text added: "old: 138.195335 142.10256"

Commit message: Version 0.1.14 - Various changes, see changelog
Signed-off-by: ray33ee <30669752+ray33ee@users.noreply.github.com>
Parts:
- moved R1 2.00 mm to (151.0, 131.9)
- moved R2 2.00 mm to (166.5, 133.8)
- moved R3 2.00 mm to (151.0, 134.3)
Routing:
- net /R: track 2.61 -> 4.61 mm
- net /B: track 2.60 -> 4.60 mm
- net /G: track 3.51 -> 5.51 mm
- net /LED_Red: track 16.8 -> 14.8 mm
- net /LED_Green: track 30.4 -> 31.1 mm
- net +5V: vias 1 -> 2
Other:
- board text removed: "old: 138.195335 142.10256"

Commit message: Version 0.1.15 - Various changes, see changelog
Signed-off-by: ray33ee <30669752+ray33ee@users.noreply.github.com>
Parts:
- moved J3 6.85 mm to (154.3, 150.0), turned to 90 degrees
- moved J2 0.90 mm to (178.2, 128.8)
Routing:
- net +3V3: track 62.4 -> 58.6 mm
- net /SDA: track 52.1 -> 49.0 mm
- net /LED_Green: track 31.1 -> 33.3 mm
- net /LED_Blue: track 17.7 -> 15.7 mm, vias 2 -> 1
- net +5V: track 40.1 -> 41.1 mm
- net GND: track 86.2 -> 85.3 mm, vias 0 -> 1
Other:
- board text added: "JLCJLCJLCJLC"
- board text added: "Valve Controller Top v1.1 William RJ Cooper github.com/ray33ee"
