File: Front/front/front.kicad_pcb (KiCad board)
At the start: 2 copper layers, 28.5 x 51.8 mm, 14 parts, among them J1 Conn_01x10_Male, J2 JST 1mm Connector, SW1 SW_Push, U1 L293D

Commit message: Version 0.1.5 - Various changes, see changelog
Signed-off-by: ray33ee <30669752+ray33ee@users.noreply.github.com>
Other:
- board text added: "Valve Controller Front v1.1|William RJ Cooper|github.com/ray33ee"
- board text removed: "Valve Controller Front v1.0|William RJ Cooper|github.com/ray33ee"

Commit message: Version 0.1.7 - Various changes, see changelog
Signed-off-by: ray33ee <30669752+ray33ee@users.noreply.github.com>
Parts:
- JP1: value SolderJumper_3_Open -> SolderJumper_3_Bridged12; footprint Jumper:SolderJumper-3_P1.3mm_Open_RoundedPad1.0x1.5mm_NumberLabels -> Jumper:SolderJumper-3_P1.3mm_Bridged12_RoundedPad1.0x1.5mm_NumberLabels
- turned JP1 to 180 degrees
Connections:
- JP1 pad 1: /Enable_High -> /Enable_Controlled
- JP1 pad 3: /Enable_Controlled -> /Enable_High
Changed lines of the file:
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@@
   (general
     (thickness 1.6)
-    (drawings 6)
+    (drawings 7)
     (tracks 279)
     (zones 0)
@@
     (add_net /Motor_Supply_Pre)
   )
+  (module Jumper:SolderJumper-3_P1.3mm_Bridged12_RoundedPad1.0x1.5mm_NumberLabels (layer F.Cu)
+    (at 206.1 92.2 180)
+    (descr "SMD Solder 3-pad Jumper, 1x1.5mm rounded Pads, 0.3mm gap, pads 1-2 bridged with 1 copper strip, labeled with numbers")
+    (tags "solder jumper open")
+    (attr virtual)
+    (fp_text reference JP1 (at 0 -1.8) (layer F.SilkS)
+      (effects (font (size 1 1) (thickness 0.15)))
+    )
+    (fp_text value SolderJumper_3_Bridged12 (at 0 1.9) (layer F.Fab) hide
+      (effects (font (size 1 1) (thickness 0.15)))
+    )
+    (fp_poly (pts (xy -0.9 -0.3) (xy -0.4 -0.3) (xy -0.4 0.3) (xy -0.9 0.3)) (layer F.Cu) (width 0))
+    (fp_line (start 2.3 1.25) (end -2.3 1.25) (layer F.CrtYd) (width 0.05))
+    (fp_line (start 2.3 1.25) (end 2.3 -1.25) (layer F.CrtYd) (width 0.05))
+    (fp_line (start -2.3 -1.25) (end -2.3 1.25) (layer F.CrtYd) (width 0.05))
+    (fp_line (start -2.3 -1.25) (end 2.3 -1.25) (layer F.CrtYd) (width 0.05))
+    (fp_line (start -1.4 -1) (end 1.4 -1) (layer F.SilkS) (width 0.12))
+    (fp_line (start 2.05 -0.3) (end 2.05 0.3) (layer F.SilkS) (width 0.12))
+    (fp_line (start 1.4 1) (end -1.4 1) (layer F.SilkS) (width 0.12))
+    (fp_line (start -2.05 0.3) (end -2.05 -0.3) (layer F.SilkS) (width 0.12))
+    (fp_arc (start -1.35 -0.3) (end -1.35 -1) (angle -90) (layer F.SilkS) (width 0.12))
+    (fp_arc (start -1.35 0.3) (end -2.05 0.3) (angle -90) (layer F.SilkS) (width 0.12))
+    (fp_arc (start 1.35 0.3) (end 1.35 1) (angle -90) (layer F.SilkS) (width 0.12))
+    (fp_arc (start 1.35 -0.3) (end 2.05 -0.3) (angle -90) (layer F.SilkS) (width 0.12))
+    (fp_text user 1 (at -2.6 0) (layer F.SilkS)
+      (effects (font (size 1 1) (thickness 0.15)))
+    )
+    (fp_text user 3 (at 2.6 0) (layer F.SilkS)
+      (effects (font (size 1 1) (thickness 0.15)))
+    )
+    (pad 1 smd custom (at -1.3 0 180) (size 1 0.5) (layers F.Cu F.Mask)
+      (net 16 /Enable_Controlled) (zone_connect 2)
+      (options (clearance outline) (anchor rect))
+      (primitives
+        (gr_poly (pts
+           (xy 0.55 -0.75) (xy 0 -0.75) (xy 0 0.75) (xy 0.55 0.75)) (width 0))
+        (gr_circle (center 0 0.25) (end 0.5 0.25) (width 0))
+        (gr_circle (center 0 -0.25) (end 0.5 -0.25) (width 0))
+      ))
+    (pad 2 smd rect (at 0 0 180) (size 1 1.5) (layers F.Cu F.Mask)
+      (net 5 /Enable))
+    (pad 3 smd custom (at 1.3 0 180) (size 1 0.5) (layers F.Cu F.Mask)
+      (net 17 /Enable_High) (zone_connect 2)
+      (options (clearance outline) (anchor rect))
+      (primitives
+        (gr_circle (center 0 0.25) (end 0.5 0.25) (width 0))
+        (gr_circle (center 0 -0.25) (end 0.5 -0.25) (width 0))
+        (gr_poly (pts
+           (xy -0.55 -0.75) (xy 0 -0.75) (xy 0 0.75) (xy -0.55 0.75)) (width 0))
+      ))
+  )
   (module MountingHole:DanfossFrontPanel (layer F.Cu)
     (at 191.77 131.78)
@@
     (pad "" np_thru_hole circle (at 5 -0.5) (size 1 1) (drill 1) (layers *.Cu *.Mask))
     (pad "" np_thru_hole circle (at 23.65 -0.5) (size 1 1) (drill 1) (layers *.Cu *.Mask))
-  )
-  (module Jumper:SolderJumper-3_P1.3mm_Open_RoundedPad1.0x1.5mm_NumberLabels (layer F.Cu)
-    (at 206.1 92.2)
-    (descr "SMD Solder 3-pad Jumper, 1x1.5mm rounded Pads, 0.3mm gap, open, labeled with numbers")
-    (tags "solder jumper open")
-    (attr virtual)
-    (fp_text reference JP1 (at 0 -1.8) (layer F.SilkS)
-      (effects (font (size 1 1) (thickness 0.15)))
-    )
-    (fp_text value SolderJumper_3_Open (at 0 1.9) (layer F.Fab) hide
-      (effects (font (size 1 1) (thickness 0.15)))
-    )
-    (fp_line (start 2.3 1.25) (end -2.3 1.25) (layer F.CrtYd) (width 0.05))
-    (fp_line (start 2.3 1.25) (end 2.3 -1.25) (layer F.CrtYd) (width 0.05))
-    (fp_line (start -2.3 -1.25) (end -2.3 1.25) (layer F.CrtYd) (width 0.05))
-    (fp_line (start -2.3 -1.25) (end 2.3 -1.25) (layer F.CrtYd) (width 0.05))
-    (fp_line (start -1.4 -1) (end 1.4 -1) (layer F.SilkS) (width 0.12))
-    (fp_line (start 2.05 -0.3) (end 2.05 0.3) (layer F.SilkS) (width 0.12))
-    (fp_line (start 1.4 1) (end -1.4 1) (layer F.SilkS) (width 0.12))
-    (fp_line (start -2.05 0.3) (end -2.05 -0.3) (layer F.SilkS) (width 0.12))
-    (fp_text user 3 (at 2.6 0) (layer F.SilkS)
-      (effects (font (size 1 1) (thickness 0.15)))
-    )
-    (fp_text user 1 (at -2.6 0) (layer F.SilkS)
-      (effects (font (size 1 1) (thickness 0.15)))
-    )
-    (fp_arc (start 1.35 -0.3) (end 2.05 -0.3) (angle -90) (layer F.SilkS) (width 0.12))
-    (fp_arc (start 1.35 0.3) (end 1.35 1) (angle -90) (layer F.SilkS) (width 0.12))
-    (fp_arc (start -1.35 0.3) (end -2.05 0.3) (angle -90) (layer F.SilkS) (width 0.12))
-    (fp_arc (start -1.35 -0.3) (end -1.35 -1) (angle -90) (layer F.SilkS) (width 0.12))
-    (pad 1 smd custom (at -1.3 0) (size 1 0.5) (layers F.Cu F.Mask)
-      (net 17 /Enable_High) (zone_connect 2)
-      (options (clearance outline) (anchor rect))
-      (primitives
-        (gr_circle (center 0 0.25) (end 0.5 0.25) (width 0))
-        (gr_circle (center 0 -0.25) (end 0.5 -0.25) (width 0))
-        (gr_poly (pts
-           (xy 0.55 -0.75) (xy 0 -0.75) (xy 0 0.75) (xy 0.55 0.75)) (width 0))
-      ))
-    (pad 3 smd custom (at 1.3 0) (size 1 0.5) (layers F.Cu F.Mask)
-      (net 16 /Enable_Controlled) (zone_connect 2)
-      (options (clearance outline) (anchor rect))
-      (primitives
-        (gr_circle (center 0 0.25) (end 0.5 0.25) (width 0))
-        (gr_circle (center 0 -0.25) (end 0.5 -0.25) (width 0))
-        (gr_poly (pts
-           (xy -0.55 -0.75) (xy 0 -0.75) (xy 0 0.75) (xy -0.55 0.75)) (width 0))
-      ))
-    (pad 2 smd rect (at 0 0) (size 1 1.5) (layers F.Cu F.Mask)
-      (net 5 /Enable))
   )
   (module Capacitor_SMD:C_1206_3216Metric_Pad1.33x1.80mm_HandSolder (layer F.Cu)
@@
     )
   )
+  (gr_poly (pts (xy 208.55 109.85) (xy 208.55 131) (xy 203.55 131) (xy 203.55 108.7) (xy 207.75 108.7)) (layer B.Mask) (width 0.1))
   (gr_text JLCJLCJLCJLC (at 206.3 131.1) (layer B.SilkS)
     (effects (font (size 1 1) (thickness 0.2)) (justify mirror))

Commit message: Version 0.1.15 - Various changes, see changelog
Signed-off-by: ray33ee <30669752+ray33ee@users.noreply.github.com>
Parts:
- added REF**: MountingHole_2.1mm, MountingHole:MountingHole_2.1mm, F.Cu at (209.0, 132.0)
- added REF**: MountingHole_2.1mm, MountingHole:MountingHole_2.1mm, F.Cu at (208.0, 132.0)
- added REF**: MountingHole_2.1mm, MountingHole:MountingHole_2.1mm, F.Cu at (207.0, 132.0)
- added REF**: MountingHole_2.1mm, MountingHole:MountingHole_2.1mm, F.Cu at (206.0, 132.0)
- added REF**: MountingHole_2.1mm, MountingHole:MountingHole_2.1mm, F.Cu at (205.0, 132.0)
- added REF**: MountingHole_2.1mm, MountingHole:MountingHole_2.1mm, F.Cu at (204.0, 132.0)
- added REF**: MountingHole_2.1mm, MountingHole:MountingHole_2.1mm, F.Cu at (203.0, 132.0)
- added REF**: PinHeader_1x04_P2.00mm_Vertical, Connector_PinHeader_2.00mm:PinHeader_1x04_P2.00mm_Vertical, F.Cu at (203.0, 142.8)
- added REF**: PinHeader_1x04_P2.00mm_Vertical, Connector_PinHeader_2.00mm:PinHeader_1x04_P2.00mm_Vertical, F.Cu at (203.0, 133.8)
- R1: footprint Resistor_THT:R_Axial_DIN0204_L3.6mm_D1.6mm_P5.08mm_Horizontal -> Resistor_THT:R_Axial_DIN0204_L3.6mm_D1.6mm_P7.62mm_Horizontal
- moved R1 2.42 mm to (195.6, 85.2)
Routing:
- net (no net): track 0.00 -> 36.0 mm
- net /Diff_P2: track 16.3 -> 12.1 mm, vias 2 -> 1
- net /Enable_Controlled: track 12.8 -> 15.9 mm
- net /Coil_B2: track 41.0 -> 43.7 mm
Other:
- board size 28.5 x 51.8 mm -> 28.5 x 64.8 mm
- board text added: "Valve Controller Front v1.2|William RJ Cooper|github.com/ray33ee"
- board text removed: "Valve Controller Front v1.1|William RJ Cooper|github.com/ray33ee"

Commit message: Version 0.1.16 - Various changes, see changelog
Signed-off-by: ray33ee <30669752+ray33ee@users.noreply.github.com>
Parts:
- removed the REF** at (209.0, 132.0)
- removed the REF** at (208.0, 132.0)
- removed the REF** at (207.0, 132.0)
- removed the REF** at (206.0, 132.0)
- removed the REF** at (205.0, 132.0)
- removed the REF** at (204.0, 132.0)
- removed the REF** at (203.0, 132.0)
- removed the REF** at (203.0, 142.8)
- removed the REF** at (203.0, 133.8)
- D1, D2: footprint Diode_SMD:D_T-1_P5.08mm_Horizontal_SurfaceMount -> Diode_SMD:D_MiniMELF
- R1: footprint Resistor_THT:R_Axial_DIN0204_L3.6mm_D1.6mm_P7.62mm_Horizontal -> Resistor_SMD:R_1206_3216Metric_Pad1.30x1.75mm_HandSolder
- moved D2 3.88 mm to (203.8, 85.4)
- moved R1 3.84 mm to (195.2, 89.0)
- moved D1 3.14 mm to (210.8, 85.1)
Routing:
- net (no net): track 36.0 -> 0.00 mm
- net +5V: track 77.2 -> 81.7 mm
- net /Diff_P2: track 12.1 -> 16.3 mm
- net /Motor_Supply_Pre: track 71.6 -> 73.4 mm, vias 3 -> 4
Other:
- board size 28.5 x 64.8 mm -> 28.5 x 51.8 mm
